File: HDK/MecatronPDU-LV.kicad_sch (KiCad schematic)
At the start: 21 parts, among them J101 Power In, J102 E-Stops, K101 Relay_SPST-NO

Commit message: updated prod
Parts:
- C101, C102, C103, C104, C105, C106, C107, C108: footprint CP_Radial_D10.0mm_P5.00mm -> lib:CP_Radial_D10.0mm_P5.00mm; sourcing-part-num (none) -> EEUFR1V561; sourcing-remarks (none) -> or any 560uF 35V cap, D10mm P5mm
- D101: footprint D_DO-35_SOD27_P7.62mm_Horizontal -> lib:D_DO-35_SOD27_P7.62mm_Horizontal; sourcing-part-num (none) -> 1N4007
- D102: value LED -> Blue LED; footprint LED_D5.0mm -> lib:LED_D5.0mm; sourcing-remarks (none) -> any blue LED, 5mm
- D103: value LED -> Green LED; footprint LED_D5.0mm -> lib:LED_D5.0mm; sourcing-remarks (none) -> any green LED, 5mm
- F101: footprint FUSE-MCCQ-122 -> lib:FUSE-MCCQ-122; sourcing-part-num (none) -> MCCQ-122
- H101, H102, H103, H104: footprint MountingHole_5.3mm_M5_ISO7380_Pad_TopBottom -> lib:MountingHole_5.3mm_M5_ISO7380_Pad_TopBottom
- J101: footprint AMASS_XT60PW-M_1x02_P7.20mm_Horizontal -> lib:AMASS_XT60PW-M_1x02_P7.20mm_Horizontal
- J102: footprint PinHeader_2x03_P2.54mm_Vertical -> lib:PinHeader_2x03_P2.54mm_Vertical
- K101: footprint G8PM1AW7RDC12 -> lib:G8PM1AW7RDC12; sourcing-part-num (none) -> G8PM-1AW7RDC12
- R101, R102: footprint R_Axial_DIN0204_L3.6mm_D1.6mm_P5.08mm_Horizontal -> lib:R_Axial_DIN0204_L3.6mm_D1.6mm_P5.08mm_Horizontal; sourcing-remarks (none) -> any 2kOhm resistor, L3.6mm
