File: HDK/Outputs.kicad_sch (KiCad schematic)
At the start: 13 parts, among them J201 V_{HV}, J202 V, J203 V, J204 V, J205 V_{SBC}, U201 TPS5460 康威科技, U202 TPS5460 康威科技, U203 TPS5460 康威科技, U204 TPS5460 康威科技

Commit message: updated prod
Parts:
- C205, C206, C207, C208: sourcing-part-num (none) -> EEUFR1V561
- J201: footprint JST_XH_B2B-XH-AM_1x02_P2.50mm_Vertical -> lib:JST_XH_B2B-XH-AM_1x02_P2.50mm_Vertical; sourcing-part-num (none) -> JST XH B2B
- J202, J203, J204: footprint PinHeader_2x05_P2.54mm_Vertical -> lib:PinHeader_2x05_P2.54mm_Vertical
- J205: footprint AMASS_XT30U-M_1x02_P5.0mm_Vertical -> lib:AMASS_XT30U-M_1x02_P5.0mm_Vertical
- U201, U202, U203, U204: footprint TPS5460 康威科技 -> lib:TPS5460 康威科技; sourcing-part-num (none) -> TPS5460 康威科技 (taobao)
Changed lines of the file:
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@@
 			)
 		)
-		(property "Footprint" "TPS5460 康威科技"
+		(property "Footprint" "lib:TPS5460 康威科技"
 			(at 76.2 76.2 0)
 			(effects
@@
 			)
 		)
+		(property "sourcing-part-num" "TPS5460 康威科技 (taobao)"
+			(at 76.2 76.2 0)
+			(effects
+				(font
+					(size 1.27 1.27)
+				)
+				(hide yes)
+			)
+		)
+		(property "sourcing-remarks" ""
+			(at 76.2 76.2 0)
+			(effects
+				(font
+					(size 1.27 1.27)
+				)
+				(hide yes)
+			)
+		)
 		(pin "EN"
 		)
@@
 			)
 		)
-		(property "Footprint" "TPS5460 康威科技"
+		(property "Footprint" "lib:TPS5460 康威科技"
 			(at 77.47 49.53 0)
 			(effects
@@
 			)
 		)
+		(property "sourcing-part-num" "TPS5460 康威科技 (taobao)"
+			(at 77.47 49.53 0)
+			(effects
+				(font
+					(size 1.27 1.27)
+				)
+				(hide yes)
+			)
+		)
+		(property "sourcing-remarks" ""
+			(at 77.47 49.53 0)
+			(effects
+				(font
+					(size 1.27 1.27)
+				)
+				(hide yes)
+			)
+		)
 		(pin "EN"
 		)
@@
 			)
 		)
+		(property "sourcing-part-num" "EEUFR1V561"
+			(at 48.26 53.34 0)
+			(effects
+				(font
+					(size 1.27 1.27)
+				)
+				(hide yes)
+			)
+		)
+		(property "sourcing-remarks" ""
+			(at 48.26 53.34 0)
+			(effects
+				(font
+					(size 1.27 1.27)
+				)
+				(hide yes)
+			)
+		)
 		(pin "2"
 		)
@@
 			)
 		)
-		(property "Footprint" "PinHeader_2x05_P2.54mm_Vertical"
+		(property "Footprint" "lib:PinHeader_2x05_P2.54mm_Vertical"
 			(at 127 31.75 0)
 			(effects
@@
 			)
 		)
+		(property "sourcing-remarks" ""
+			(at 127 31.75 0)
+			(effects
+				(font
+					(size 1.27 1.27)
+				)
+				(hide yes)
+			)
+		)
 		(pin "4"
 		)
@@
 			)
 		)
-		(property "Footprint" "JST_XH_B2B-XH-AM_1x02_P2.50mm_Vertical"
+		(property "Footprint" "lib:JST_XH_B2B-XH-AM_1x02_P2.50mm_Vertical"
 			(at 127 17.78 0)
 			(effects
@@
 			)
 		)
+		(property "sourcing-part-num" "JST XH B2B"
+			(at 127 17.78 0)
+			(effects
+				(font
+					(size 1.27 1.27)
+				)
+				(hide yes)
+			)
+		)
+		(property "sourcing-remarks" ""
+			(at 127 17.78 0)
+			(effects
+				(font
+					(size 1.27 1.27)
+				)
+				(hide yes)
+			)
+		)
 		(pin "2"
 		)
@@
 			)
 		)
+		(property "sourcing-part-num" "EEUFR1V561"
+			(at 88.9 80.01 0)
+			(effects
+				(font
+					(size 1.27 1.27)
+				)
+				(hide yes)
+			)
+		)
+		(property "sourcing-remarks" ""
+			(at 88.9 80.01 0)
+			(effects
+				(font
+					(size 1.27 1.27)
+				)
+				(hide yes)
+			)
+		)
 		(pin "2"
 		)
@@
 			)
 		)
-		(property "Footprint" "AMASS_XT30U-M_1x02_P5.0mm_Vertical"
+		(property "Footprint" "lib:AMASS_XT30U-M_1x02_P5.0mm_Vertical"
 			(at 125.73 78.74 0)
 			(effects
@@
 			)
 		)
+		(property "sourcing-remarks" ""
+			(at 125.73 78.74 0)
+			(effects
+				(font
+					(size 1.27 1.27)
+				)
+				(hide yes)
+			)
+		)
 		(pin "1"
 		)
@@
 			)
 		)
+		(property "sourcing-part-num" "EEUFR1V561"
+			(at 46.99 80.01 0)
+			(effects
+				(font
+					(size 1.27 1.27)
+				)
+				(hide yes)
+			)
+		)
+		(property "sourcing-remarks" ""
+			(at 46.99 80.01 0)
+			(effects
+				(font
+					(size 1.27 1.27)
+				)
+				(hide yes)
+			)
+		)
 		(pin "2"
 		)
@@
 			)
 		)
-		(property "Footprint" "PinHeader_2x05_P2.54mm_Vertical"
+		(property "Footprint" "lib:PinHeader_2x05_P2.54mm_Vertical"
 			(at 127 64.77 0)
 			(effects
@@
 			)
 		)
+		(property "sourcing-remarks" ""
+			(at 127 64.77 0)
+			(effects
+				(font
+					(size 1.27 1.27)
+				)
+				(hide yes)
+			)
+		)
 		(pin "4"
 		)
@@
 			)
 		)
-		(property "Footprint" "PinHeader_2x05_P2.54mm_Vertical"
+		(property "Footprint" "lib:PinHeader_2x05_P2.54mm_Vertical"
 			(at 127 48.26 0)
 			(effects
@@
 			)
 		)
+		(property "sourcing-remarks" ""
+			(at 127 48.26 0)
+			(effects
+				(font
+					(size 1.27 1.27)
+				)
+				(hide yes)
+			)
+		)
 		(pin "4"
 		)
@@
 			)
 		)
-		(property "Footprint" "TPS5460 康威科技"
+		(property "Footprint" "lib:TPS5460 康威科技"
 			(at 34.29 76.2 0)
 			(effects
@@
 			)
 		)
+		(property "sourcing-part-num" "TPS5460 康威科技 (taobao)"
+			(at 34.29 76.2 0)
+			(effects
+				(font
+					(size 1.27 1.27)
+				)
+				(hide yes)
+			)
+		)
+		(property "sourcing-remarks" ""
+			(at 34.29 76.2 0)
+			(effects
+				(font
+					(size 1.27 1.27)
+				)
+				(hide yes)
+			)
+		)
 		(pin "EN"
 		)
@@
 			)
 		)
-		(property "Footprint" "TPS5460 康威科技"
+		(property "Footprint" "lib:TPS5460 康威科技"
 			(at 35.56 49.53 0)
 			(effects
@@
 			)
 		)
+		(property "sourcing-part-num" "TPS5460 康威科技 (taobao)"
+			(at 35.56 49.53 0)
+			(effects
+				(font
+					(size 1.27 1.27)
+				)
+				(hide yes)
+			)
+		)
+		(property "sourcing-remarks" ""
+			(at 35.56 49.53 0)
+			(effects
+				(font
+					(size 1.27 1.27)
+				)
+				(hide yes)
+			)
+		)
 		(pin "EN"
 		)
@@
 			(at 90.17 53.34 0)
 			(effects
+				(font
+					(size 1.27 1.27)
+				)
+				(hide yes)
+			)
+		)
+		(property "sourcing-part-num" "EEUFR1V561"
+			(at 90.17 53.34 0)
+			(effects
+				(font
+					(size 1.27 1.27)
+				)
+				(hide yes)
+			)
+		)
+		(property "sourcing-remarks" ""
+			(at 90.17 53.34 0)
+			(effects
